File: schematics/ESP32 adon V2/ESP32 adon V2.kicad_sch (KiCad schematic)
At the start: 38 parts, among them J1 Conn_01x08_Pin, J2 Conn_01x08_Pin, J3 Conn_01x02_Pin, J4 Conn_01x08_Pin, J5 Conn_01x08_Pin, J6 USB4215-03-A_REVA, J7 Conn_01x04_Pin, J8 Conn_01x02_Socket, Q4 MMBT7002K, Q5 MMBT7002K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

Commit message: verbeterde pcb layout
Parts:
- removed J8: Conn_01x02_Socket, Connector_PinSocket_1.27mm:PinSocket_2x01_P1.27mm_Vertical, symbol Connector:Conn_01x02_Socket
- added J8: Conn_01x02_Pin, Resistor_SMD:R_0603_1608Metric_Pad0.98x0.95mm_HandSolder, symbol Connector:Conn_01x02_Pin
Connections:
- net D+: now also J8.2 (Pin_2)
- net D-: now also J8.1 (Pin_1)
- net GND: now also D3.1; no longer MT1.10 (RESV), MT1.11 (RESV), MT1.2 (RESV), MT1.3 (RESV)
- net Vin_reg: now reaches C3.1, D1.1 (K), D2.1 (K), U4.1 (IN), U4.3 (EN)
- net at J4.1 (Pin_1): now also U1.19 (GPIO21); no longer U1.16 (GPIO18)
- net at J4.2 (Pin_2): now also U1.18 (GPIO20); no longer U1.17 (GPIO19)
- net at J4.3 (Pin_3): now also U1.17 (GPIO19); no longer U1.18 (GPIO20)
- net at J4.4 (Pin_4): now also U1.16 (GPIO18); no longer U1.19 (GPIO21)
- new net: MT1.10 (RESV), MT1.11 (RESV), MT1.2 (RESV), MT1.3 (RESV)
