File: schematics/ESP32 adon V3/ESP32 adon V3.kicad_sch (KiCad schematic)
At the start: 38 parts, among them J1 Conn_01x08_Pin, J2 Conn_01x08_Pin, J3 Conn_01x02_Pin, J4 Conn_01x08_Pin, J5 Conn_01x08_Pin, J6 USB4215-03-A_REVA, J7 Conn_01x04_Pin, J8 Conn_01x02_Pin, Q4 MMBT7002K, Q5 MMBT7002K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

Commit message: update de schematics
Parts:
- removed D3: SMF05C.TCT, Package_TO_SOT_SMD:Vishay_PowerPAK_SC70-6L_Dual, symbol SMF05C.TCT:SMF05C.TCT
- removed Q4, Q5, Q6: MMBT7002K, Package_TO_SOT_SMD:SOT-23, symbol Simulation_SPICE:NMOS
- added Q1, Q2, Q3: MMBT7001K, Package_TO_SOT_SMD:TSOT-23, symbol Simulation_SPICE:NMOS
- added U5: USBLC6-2SC6, Package_TO_SOT_SMD:SOT-23-6, symbol Power_Protection:USBLC6-2SC6
Connections:
- net +3.3V: now also Q1.1 (G), Q2.1 (G), Q3.1 (G)
- net +5Vin: now also U5.5 (VBUS)
- net D+: now also U5.4 (I/O2); no longer J6.A6 (DP1), J6.B6 (DP2)
- net D-: now also U5.6 (I/O1); no longer J6.A7 (DN1), J6.B7 (DN2)
- net GND: now also U5.2 (GND)
- net SCL_{3.3V}: now also Q3.2 (S)
- net SCL_{5V}: now also Q3.3 (D)
- net SDA_{3.3V}: now also Q2.2 (S)
- net SDA_{5V}: now also Q2.3 (D)
- net TX: now also Q1.3 (D)
- net at R8.2, U1.25 (U0TXD/GPIO16): now also Q1.2 (S)
- new net: J6.A7 (DN1), J6.B7 (DN2), U5.1 (I/O1)
- new net: J6.A6 (DP1), J6.B6 (DP2), U5.3 (I/O2)

Commit message: begin al met het tekenen van ESP32 addon V3
Parts:
- removed J8: Conn_01x02_Pin, Resistor_SMD:R_0603_1608Metric_Pad0.98x0.95mm_HandSolder, symbol Connector:Conn_01x02_Pin
- added J10, J11, J12, J13, J14: Conn_01x01, Connector_Wire:SolderWirePad_1x01_SMD_1x2mm, symbol Connector_Generic:Conn_01x01
- added J9: Conn_01x04_Pin, Connector_PinSocket_2.54mm:PinSocket_1x04_P2.54mm_Vertical, symbol Connector:Conn_01x04_Pin
Connections:
- net +3.3V: now also J9.1 (Pin_1)
- net GND: now also J9.4 (Pin_4)
- net SCL_{3.3V}: now also J9.2 (Pin_2)
- net SDA_{3.3V}: now also J9.3 (Pin_3)
- net at MT1.4 (INT1/INT): now also J13.1 (Pin_1)
- net at MT1.9 (INT2): now also J14.1 (Pin_1)
- net at U6.4 (INT/TRG): now also J12.1 (Pin_1)
- net at U3.2 (ALERT/RDY): now also J11.1 (Pin_1)
- net at U2.1 (~{INT}): now also J10.1 (Pin_1)
- no-connect marks 26 -> 21

Commit message: verder tekenen en datasheets controleren
Connections:
- net GND: now also U6.3 (MISO)
- no-connect marks 21 -> 20
Changed lines of the file:
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@@
+	)
+	(junction
+		(at 97.79 81.28)
+		(diameter 0)
+		(color 0 0 0 1)
 	)
 	(junction
@@
 	)
 	(no_connect
-		(at 101.6 76.2)
-	)
-	(no_connect
 		(at 58.42 34.29)
 	)
@@
 	(wire
 		(pts
+			(xy 97.79 81.28) (xy 97.79 76.2)
+		)
+		(stroke
+			(width 0)
+			(type default)
+			(color 0 0 0 1)
+		)
+	)
+	(wire
+		(pts
 			(xy 254 68.58) (xy 266.7 68.58)
 		)
@@
 	(wire
 		(pts
-			(xy 83.82 81.28) (xy 101.6 81.28)
+			(xy 83.82 81.28) (xy 97.79 81.28)
 		)
 		(stroke
@@
 	(wire
 		(pts
+			(xy 97.79 76.2) (xy 101.6 76.2)
+		)
+		(stroke
+			(width 0)
+			(type default)
+			(color 0 0 0 1)
+		)
+	)
+	(wire
+		(pts
 			(xy 115.57 106.68) (xy 115.57 107.95)
 		)
@@
 		)
 		(stroke
+			(width 0)
+			(type default)
+			(color 0 0 0 1)
+		)
+	)
+	(wire
+		(pts
+			(xy 97.79 81.28) (xy 101.6 81.28)
+		)
+		(stroke
