File: schematics/lijnsensor V2 met IO_expander/lijnsensor V2 met IO_expander.kicad_sch (KiCad schematic)
At the start: 32 parts, among them J2 Conn_01x05_Pin, U1 USBLC6-2SC6, U10 AS7343xDLG, U11 AS7343xDLG, U12 TCA9535RGER, U2 TCA9548ARGER, U3 TLV75718PDBV, U4 AS7343xDLG, U5 AS7343xDLG, U6 AS7343xDLG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

Commit message: begin al met het toevoegen van de io extender nog niet klaar
Parts:
- added H1, H2, H3, H4: MountingHole, MountingHole:MountingHole_4.3mm_M4, symbol Mechanical:MountingHole
- added H5, H6: MountingHole, MountingHole:MountingHole_8.4mm_M8, symbol Mechanical:MountingHole
- U12: footprint Package_DFN_QFN:VQFN-24-1EP_4x4mm_P0.5mm_EP2.45x2.45mm -> Package_DFN_QFN:Texas_RGE0024H_VQFN-24-1EP_4x4mm_P0.5mm_EP2.7x2.7mm
- U2: footprint Package_DFN_QFN:Texas_RGE0024C_VQFN-24-1EP_4x4mm_P0.5mm_EP2.1x2.1mm -> Package_DFN_QFN:Texas_RGE0024H_VQFN-24-1EP_4x4mm_P0.5mm_EP2.7x2.7mm
Connections:
- net GND: now also U2.25 (EPAD)
- net at U10.6 (GPIO): now also U12.7 (P06)
- net at U10.7 (INT): now also U12.16 (P16)
- net at R4.2, U4.2 (SCL): now also U2.2 (SC0); no longer U2.8 (SC3)
- net at U9.6 (GPIO): now also U12.6 (P05)
- net at U9.7 (INT): now also U12.15 (P15)
- net at R9.2, U7.8 (SDA): now also U2.7 (SD3); no longer U2.1 (SD0)
- net at U4.6 (GPIO): now also U12.1 (P00)
- net at U4.7 (INT): now also U12.10 (P10)
- net at R3.2, U4.8 (SDA): now also U2.1 (SD0); no longer U2.7 (SD3)
- net at U8.6 (GPIO): now also U12.5 (P04)
- net at U8.7 (INT): now also U12.14 (P14)
- net at R6.2, U5.2 (SCL): now also U2.4 (SC1); no longer U2.6 (SC2)
- net at U5.6 (GPIO): now also U12.2 (P01)
- net at U5.7 (INT): now also U12.11 (P11)
- net at R5.2, U5.8 (SDA): now also U2.3 (SD1); no longer U2.5 (SD2)
- net at R8.2, U6.2 (SCL): now also U2.5 (SD2); no longer U2.4 (SC1)
- net at U6.6 (GPIO): now also U12.3 (P02)
- net at U6.7 (INT): now also U12.12 (P12)
- net at R7.2, U6.8 (SDA): now also U2.6 (SC2); no longer U2.3 (SD1)
- net at R10.2, U7.2 (SCL): now also U2.8 (SC3); no longer U2.2 (SC0)
- net at U7.6 (GPIO): now also U12.4 (P03)
- net at U7.7 (INT): now also U12.13 (P13)
- net at U12.17 (P17): now also U11.7 (INT)
- net at U12.8 (P07): now also U11.6 (GPIO)
- no-connect marks 24 -> 8
Other:
- moved on the sheet: R1, R10, R11, R12, R13, R14, R15, R16, R17, R2, R3, R4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
