File: schematics/hoofd nieuw V2/hoofd nieuw V2.kicad_pcb (KiCad board)
At the start: 2 copper layers, 175 x 75 mm, 44 parts, among them J1 Conn_01x04_Pin, J2 Conn_01x02_Pin, J3 SFR02, J4 Conn_01x03_Pin, J5 Conn_01x01, J6 Conn_01x01, U1 ATtiny402-SS, U2 BH1750FVI-TR, U3 BH1750FVI-TR, Y1 ECS-2333MV-100-BN-TR

Commit message: voeg mijn naam toe aan nieuw hoofd en lijnsensor
Other:
- board text added: "ontworpen door Stan Debakker"
Changed lines of the file:
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@@
 			(psa4output no)
 			(plot_black_and_white yes)
-			(plotinvisibletext no)
 			(sketchpadsonfab no)
 			(plotpadnumbers no)
@@
 		(layer "Edge.Cuts")
 	)
+	(gr_text "ontworpen door\nStan Debakker"
+		(at 121 57.5 0)
+		(layer "F.SilkS")
+		(effects
+			(font
+				(size 3 3)
+				(thickness 0.375)
+			)
+			(justify left bottom)
+		)
+	)
+	(gr_text "ontworpen door\nStan Debakker"
+		(at 157 57.5 0)
+		(layer "B.SilkS")
+		(effects
+			(font
+				(size 3 3)
+				(thickness 0.375)
+			)
+			(justify left bottom mirror)
+		)
+	)
 	(via

Commit message: maak de .gbr bestanden
Routing:
- net GND: vias 408 -> 406
Changed lines of the file:
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@@
 			(drillshape 0)
 			(scaleselection 1)
-			(outputdirectory "")
+			(outputdirectory "hoofd_nieuw_V2/")
 		)
 	)
@@
 	)
 	(via
-		(at 134.84 62.31)
-		(size 0.6)
-		(drill 0.3)
-		(layers "F.Cu" "B.Cu")
-		(free yes)
-		(net 1)
-	)
-	(via
 		(at 191 25)
 		(size 0.6)
@@
 		(size 0.6)
 		(drill 0.3)
-		(layers "F.Cu" "B.Cu")
-		(free yes)
-		(net 1)
-	)
-	(via
-		(at 206 25)
-		(size 0.6)
-		(drill 0.3)
