File: schematics/lijnsensor V2/lijnsensor V2.kicad_pcb (KiCad board)
At the start: 2 copper layers, 137 x 105 mm, 37 parts, among them J1 Conn_01x04_Pin, U1 USBLC6-2SC6, U10 AS7343xDLG, U11 AS7343xDLG, U2 TCA9548APWR, U3 TLV75718PDBV, U4 AS7343xDLG, U5 AS7343xDLG, U6 AS7343xDLG, U7 AS7343xDLG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

Commit message: maak de .gbr bestanden
Routing:
- net GND: vias 388 -> 387
Changed lines of the file:
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@@
 			(drillshape 0)
 			(scaleselection 1)
-			(outputdirectory "")
+			(outputdirectory "lijnsensor_V2/")
 		)
 	)
@@
 			(at 0 -5.3 0)
 			(layer "F.SilkS")
+			(hide yes)
 			(effects
 				(font
@@
 			(at 0 5.3 0)
 			(layer "F.Fab")
+			(hide yes)
 			(effects
 				(font
@@
 			(at 0 -9.4 0)
 			(layer "F.SilkS")
+			(hide yes)
 			(effects
 				(font
@@
 			(at 0 9.4 0)
 			(layer "F.Fab")
+			(hide yes)
 			(effects
 				(font
@@
 			(at 0 -5.3 0)
 			(layer "F.SilkS")
+			(hide yes)
 			(effects
 				(font
@@
 			(at 0 5.3 0)
 			(layer "F.Fab")
+			(hide yes)
 			(effects
 				(font
@@
 			(at 0 -5.3 0)
 			(layer "F.SilkS")
+			(hide yes)
 			(effects
 				(font
@@
 			(at 0 5.3 0)
 			(layer "F.Fab")
+			(hide yes)
 			(effects
 				(font
@@
 			(at 0 -5.3 0)
 			(layer "F.SilkS")
+			(hide yes)
 			(effects
 				(font
@@
 			(at 0 5.3 0)
 			(layer "F.Fab")
+			(hide yes)
 			(effects
 				(font
@@
 			(at 0 -9.4 0)
 			(layer "F.SilkS")
+			(hide yes)
 			(effects
 				(font
@@
 			(at 0 9.4 0)
 			(layer "F.Fab")
+			(hide yes)
 			(effects
 				(font
@@
 	)
 	(segment
+		(start 90.451827 74.3)
+		(end 90.557659 74.3)
+		(width 0.3)
+		(layer "F.Cu")
+		(net 3)
+	)
+	(segment
+		(start 98.405832 66.451827)
+		(end 90.557659 74.3)
+		(width 0.3)
+		(layer "F.Cu")
+		(net 3)
+	)
+	(segment
 		(start 56.638 137.587)
 		(end 57.025 137.2)
@@
 	)
 	(segment
-		(start 58.45776 135.76724)
-		(end 58.45776 106.294067)
+		(start 100.748173 66.451827)
+		(end 98.405832 66.451827)
 		(width 0.3)
 		(layer "F.Cu")
@@
 	)
 	(segment
-		(start 58.45776 106.294067)
-		(end 98.3 66.451827)
+		(start 115.1375 59.625)
+		(end 107.575 59.625)
 		(width 0.3)
 		(layer "F.Cu")
@@
 	)
 	(segment
-		(start 56.638 138.8)
-		(end 56.638 137.587)
+		(start 107.575 59.625)
+		(end 100.748173 66.451827)
 		(width 0.3)
 		(layer "F.Cu")
@@
 	)
 	(segment
-		(start 98.3 66.451827)
-		(end 100.748173 66.451827)
+		(start 58.45776 135.76724)
+		(end 58.45776 106.294067)
 		(width 0.3)
 		(layer "F.Cu")
@@
 	)
 	(segment
-		(start 100.748173 66.451827)
-		(end 107.575 59.625)
+		(start 56.638 138.8)
+		(end 56.638 137.587)
 		(width 0.3)
 		(layer "F.Cu")
@@
 	)
 	(segment
-		(start 107.575 59.625)
-		(end 115.1375 59.625)
+		(start 58.45776 106.294067)
+		(end 90.451827 74.3)
 		(width 0.3)
 		(layer "F.Cu")
@@
 	)
 	(via
-		(at 143 72.5)
-		(size 0.6)
-		(drill 0.3)
-		(layers "F.Cu" "B.Cu")
-		(free yes)
-		(net 5)
-	)
-	(via
 		(at 80.5 77.5)
 		(size 0.6)
@@
 	)
 	(segment
-		(start 53.8 141.2)
-		(end 53.8 140.425)
+		(start 55.85 143.25)
+		(end 53.8 141.2)
+		(width 0.3)
+		(layer "F.Cu")
+		(net 17)
+	)
+	(segment
+		(start 58.03 143.25)
+		(end 55.85 143.25)
 		(width 0.3)
 		(layer "F.Cu")
@@
 	)
 	(segment
-		(start 58.95876 106.501587)
-		(end 58.95876 142.32124)
+		(start 58.95876 142.32124)
+		(end 58.03 143.25)
 		(width 0.3)
 		(layer "F.Cu")
@@
 	)
 	(segment
-		(start 54.625 139.6)
-		(end 55.362 139.6)
+		(start 115.1375 60.275)
+		(end 115.1115 60.249)
 		(width 0.3)
 		(layer "F.Cu")
@@
 	)
 	(segment
-		(start 101.047173 66.952827)
-		(end 98.50752 66.952827)
+		(start 98.613352 66.952827)
+		(end 90.765179 74.801)
 		(width 0.3)
 		(layer "F.Cu")
@@
 	)
 	(segment
-		(start 58.03 143.25)
-		(end 55.85 143.25)
+		(start 54.625 139.6)
+		(end 55.362 139.6)
 		(width 0.3)
 		(layer "F.Cu")
@@
 	)
 	(segment
-		(start 115.1375 60.275)
-		(end 115.1115 60.249)
+		(start 90.659347 74.801)
+		(end 58.95876 106.501587)
 		(width 0.3)
 		(layer "F.Cu")
@@
 	)
 	(segment
-		(start 98.50752 66.952827)
-		(end 58.95876 106.501587)
+		(start 101.047173 66.952827)
+		(end 98.613352 66.952827)
 		(width 0.3)
 		(layer "F.Cu")
@@
 	)
 	(segment
-		(start 55.85 143.25)
-		(end 53.8 141.2)
+		(start 58.95876 106.501587)
+		(end 58.95876 142.32124)
+		(width 0.3)
+		(layer "F.Cu")
+		(net 17)
+	)
+	(segment
+		(start 90.765179 74.801)
+		(end 90.659347 74.801)
 		(width 0.3)
 		(layer "F.Cu")
@@
 	)
 	(segment
-		(start 58.95876 142.32124)
-		(end 58.03 143.25)
+		(start 53.8 141.2)
+		(end 53.8 140.425)
 		(width 0.3)
 		(layer "F.Cu")
@@
 		(polygon
 			(pts
-				(xy 187 156) (xy 187 50) (xy 50 50) (xy 50 156)
+				(xy 187 156) (xy 187 51) (xy 50 51) (xy 50 156)
 			)
 		)
