File: schematics/ESP32 adon V4/ESP32 adon V4.kicad_pcb (KiCad board)
At the start: 2 copper layers, 42 x 64.6 mm, 43 parts, among them J1 Conn_01x08_Pin, J10 Conn_01x01, J11 Conn_01x01, J12 Conn_01x01, J13 Conn_01x01, J14 Conn_01x01, J2 Conn_01x08_Pin, J3 Conn_01x02_Pin, J4 Conn_01x08_Pin, J5 Conn_01x08_Pin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

Commit message: update de ESP addon en de powerpoint
Parts:
- removed U2: TCA9535DBR, Package_SO:TSSOP-24_4.4x7.8mm_P0.65mm
- added R9: 10K, Resistor_SMD:R_0603_1608Metric, F.Cu at (58.2, 53.9)
- added U7: PI4IOE5V6416, Package_SO:TSSOP-24_4.4x7.8mm_P0.65mm, F.Cu at (55.0, 58.8)
- moved J10 0.19 mm to (59.8, 56.2)
Connections:
- MT1 pad 2: GND -> unconnected-(MT1-RESV-Pad10)
- MT1 pad 3: GND -> unconnected-(MT1-RESV-Pad10)_1
Routing:
- net /SCL_{5V}: track 89.5 -> 71.9 mm, vias 10 -> 6
- net /SDA_{5V}: track 92.0 -> 75.7 mm, vias 12 -> 8
- net +3.3V: track 106.3 -> 120.4 mm
- net /SCL_{3.3V}: track 70.6 -> 78.3 mm, vias 3 -> 5
- net Net-(J1-Pin_8): track 13.0 -> 6.94 mm
- net /SDA_{3.3V}: track 78.2 -> 84.1 mm, vias 3 -> 5
- net Net-(U7-~{Reset}): track 0.00 -> 2.03 mm
- net GND: vias 262 -> 258

Commit message: werk verder aan de liberary
Routing:
- net /SCL_{5V}: track 71.9 -> 68.9 mm, vias 6 -> 4
- net /SDA_{5V}: track 75.7 -> 73.0 mm, vias 8 -> 6
- net GND: vias 258 -> 257
